Commit message: Some initial tests on ignition

File: stretch_description/urdf/stretch_main.xacro (robot description, xacro)
@@ -1,4 +1,5 @@
 <?xml version="1.0"?>
 <robot xmlns:xacro="http://www.ros.org/wiki/xacro" name="stretch_main">
+  <xacro:property name="M_PI" value="3.1415926535897931" />
   <link
     name="base_link">
@@ -48,12 +49,12 @@
         rpy="0 0 0" />
       <mass
-        value="0.00356714564938475" />
-      <inertia
-        ixx="0"
-        ixy="0"
-        ixz="0"
-        iyy="0"
-        iyz="0"
-        izz="0" />
+        value="0.01" />
+      <inertia
+        ixx="0.001"
+        ixy="0"
+        ixz="0"
+        iyy="0.001"
+        iyz="0"
+        izz="0.001" />
     </inertial>
     <visual>
@@ -81,16 +82,9 @@
     </collision>
   </link>
-  <joint
-    name="joint_right_wheel"
-    type="continuous">
-    <origin
-      xyz="-0.00300000000000034 -0.15765 0.0508000000000004"
-      rpy="-1.57079632679489 -1.11022302462516E-16 7.28583859910277E-17" />
-    <parent
-      link="base_link" />
-    <child
-      link="link_right_wheel" />
-    <axis
-      xyz="0 0 1" />
+  <joint name="joint_right_wheel" type="continuous">
+    <parent link="base_link"/>
+    <child link="link_right_wheel"/>
+    <origin xyz="-0.003 -0.15765 0.05" rpy="-1.5707963267949 0 0"/>
+    <axis xyz="0 0 1" />
   </joint>
   <link
@@ -101,12 +95,12 @@
         rpy="0 0 0" />
       <mass
-        value="0.00356714564938459" />
-      <inertia
-        ixx="0"
-        ixy="0"
-        ixz="0"
-        iyy="0"
-        iyz="0"
-        izz="0" />
+        value="0.01" />
+      <inertia
+        ixx="0.001"
+        ixy="0"
+        ixz="0"
+        iyy="0.001"
+        iyz="0"
+        izz="0.001" />
     </inertial>
     <visual>
@@ -134,16 +128,58 @@
     </collision>
   </link>
-  <joint
-    name="joint_left_wheel"
-    type="continuous">
-    <origin
-      xyz="-0.00300000000001899 0.15765 0.0507999999999994"
-      rpy="-1.5707963267949 3.16227047920818E-31 7.88745438253713E-16" />
-    <parent
-      link="base_link" />
-    <child
-      link="link_left_wheel" />
-    <axis
-      xyz="0 0 1" />
+  <joint name="joint_left_wheel" type="continuous">
+    <parent link="base_link"/>
+    <child link="link_left_wheel"/>
+    <origin xyz="-0.003 0.15765 0.05" rpy="-1.5707963267949 0 0"/>
+    <axis xyz="0 0 1" />
+  </joint>
+  <link name="caster_link">
+    <collision>
+      <geometry>
+        <sphere radius="0.032"/>
+      </geometry>
+      <origin rpy="0 0 0" xyz="0 0 0"/>
+      <surface>
+        <friction>
+          <ode>
+            <mu>0</mu>
+            <mu2>0</mu2>
+            <slip1>1.0</slip1>
+            <slip2>1.0</slip2>
+          </ode>
+        </friction>
+      </surface>
+    </collision>
+    <visual>
+      <origin
+        xyz="0 0 0"
+        rpy="0 0 0" />
+      <geometry>
+        <mesh
+          filename="package://stretch_description/meshes/omni_wheel_m.STL" />
+      </geometry>
+      <material
+        name="">
+        <color
+          rgba="0.792156862745098 0.819607843137255 0.933333333333333 1" />
+      </material>
+    </visual>
+    <inertial>
+      <mass value="0.01" />
+      <origin xyz="0 0 0" />
+      <inertia
+        ixx="0.001"
+        ixy="0"
+        ixz="0"
+        iyy="0.001"
+        iyz="0"
+        izz="0.001" />
+    </inertial>
+  </link>
+  <joint name="caster_joint" type="fixed">
+    <parent link="base_link"/>
+    <child link="caster_link"/>
+    <origin xyz="-0.245 0.0 0.032" rpy="${-M_PI/2} 0 0"/>
+    <axis xyz="0 0 1" />
   </joint>
   <link
@@ -200,5 +236,5 @@
       xyz="0 0 0" />
   </joint>
-  <link
+  <!-- <link
     name="link_lift">
     <inertial>
@@ -252,7 +288,4 @@
     <axis
 	xyz="0 0 1" />
-  <!-- for now: hand copied range_m: from lift: from ~/repos/stretch_fleet/stretch-re1-1001/stretch_re1_factory_params.yaml -->
-  <!--<limit effort="100" lower="0.0" upper="1.095" velocity="1.0"/>-->
-  <!-- copied value did not reach the top of mesh model with GUI sliders and RViz -->
   <limit effort="100" lower="0.0" upper="1.1" velocity="1.0"/>
   </joint>
@@ -319,10 +352,10 @@
         value="0.0626921047058405" />
       <inertia
-        ixx="0.000115246639451415"
-        ixy="4.42139679831176E-14"
-        ixz="1.89711279909763E-09"
-        iyy="0.000115246639420046"
-        iyz="-2.68592949587539E-09"
-        izz="9.38270676408352E-14" />
+        ixx="0.001"
+        ixy="0"
+        ixz="0"
+        iyy="0.001"
+        iyz="0"
+        izz="0.001" />
     </inertial>
     <visual>
@@ -362,5 +395,4 @@
     <axis
 	xyz="0 0 1" />
-    <!-- 0.13 = 0.52/4-->
     <limit effort="100" lower="0.0" upper="0.13" velocity="1.0"/>
   </joint>
@@ -374,10 +406,10 @@
         value="0.0569074368576238" />
       <inertia
-        ixx="0.000105206697151872"
-        ixy="2.59896259031046E-14"
-        ixz="1.69941454517918E-09"
-        iyy="0.000105206697154717"
-        iyz="-1.60895568923743E-09"
-        izz="5.20570301686304E-14" />
+        ixx="0.001"
+        ixy="0"
+        ixz="0"
+        iyy="0.001"
+        iyz="0"
+        izz="0.001" />
     </inertial>
     <visual>
@@ -417,5 +449,4 @@
     <axis
 	xyz="0 0 1" />
-    <!-- 0.13 = 0.52/4-->
     <limit effort="100" lower="0.0" upper="0.13" velocity="1.0"/>
   </joint>
@@ -429,10 +460,10 @@
         value="0.0511763619538321" />
       <inertia
-        ixx="9.58490021274768E-05"
-        ixy="2.27446667584309E-14"
-        ixz="1.54951672295709E-09"
-        iyy="9.5849002131875E-05"
-        iyz="-1.40692486873422E-09"
-        izz="4.57014633924348E-14" />
+        ixx="0.001"
+        ixy="0"
+        ixz="0"
+        iyy="0.001"
+        iyz="0"
+        izz="0.001" />
     </inertial>
     <visual>
@@ -472,5 +503,4 @@
     <axis
 	xyz="0 0 1" />
-    <!-- 0.13 = 0.52/4-->
     <limit effort="100" lower="0.0" upper="0.13" velocity="1.0"/>
   </joint>
@@ -484,10 +514,10 @@
         value="0.101241250325294" />
       <inertia
-        ixx="0.000227156999010352"
-        ixy="8.90680620109423E-06"
-        ixz="-7.91132210985695E-05"
-        iyy="0.000300732790537324"
-        iyz="7.21771824540896E-06"
-        izz="9.35784422621597E-05" />
+        ixx="0.001"
+        ixy="0"
+        ixz="0"
+        iyy="0.001"
+        iyz="0"
+        izz="0.001" />
     </inertial>
     <visual>
@@ -527,5 +557,4 @@
     <axis
 	xyz="0 0 1" />
-    <!-- 0.13 = 0.52/4-->
     <limit effort="100" lower="0.0" upper="0.13" velocity="1.0"/>
   </joint>
@@ -539,10 +568,10 @@
         value="0.0405398981326229" />
       <inertia
-        ixx="2.20062857967227E-09"
-        ixy="1.15494401227051E-13"
-        ixz="1.02598056874346E-11"
-        iyy="2.20039759185237E-09"
-        iyz="-2.47692875363392E-11"
-        izz="3.26666802416509E-13" />
+        ixx="0.001"
+        ixy="0"
+        ixz="0"
+        iyy="0.001"
+        iyz="0"
+        izz="0.001" />
     </inertial>
     <visual>
@@ -557,5 +586,5 @@
         name="">
         <color
-	  rgba="0.792156862745098 0.819607843137255 0.933333333333333 1" />
+	rgba="0.792156862745098 0.819607843137255 0.933333333333333 1" />
       </material>
     </visual>
@@ -582,10 +611,4 @@
     <axis
       xyz="0 0 -1" />
-    <!--
-	stowed to front ~225 deg: 3.15159 x 1.25 = 3.9395
-	using 4.0
-	stowed to back ~100 deg:  100 / 180 x 3.14159 = 1.7453
-	using -1.75
-    -->
     <limit effort="100" lower="-1.75" upper="4.0" velocity="1.0"/>
   </joint>
@@ -599,10 +622,10 @@
         value="0.129454717596498" />
       <inertia
-        ixx="2.9340596231093E-05"
-        ixy="-7.89638931853666E-07"
-        ixz="-4.74678128515878E-06"
-        iyy="2.68283736177377E-05"
-        iyz="1.80251508621876E-06"
-        izz="1.4617291423745E-05" />
+        ixx="0.001"
+        ixy="0"
+        ixz="0"
+        iyy="0.001"
+        iyz="0"
+        izz="0.001" />
     </inertial>
     <visual>
@@ -652,10 +675,10 @@
         value="0.035858341182617" />
       <inertia
-        ixx="2.75847937559827E-05"
-        ixy="5.25762707913649E-07"
-        ixz="-9.28796751052893E-07"
-        iyy="2.08815921106858E-05"
-        iyz="1.17265055331737E-05"
-        izz="6.78612505435872E-06" />
+        ixx="0.001"
+        ixy="0"
+        ixz="0"
+        iyy="0.001"
+        iyz="0"
+        izz="0.001" />
     </inertial>
     <visual>
@@ -695,5 +718,4 @@
     <axis
 	xyz="0 0 1" />
-    <!-- unconstrained range for now -->
     <limit effort="100" lower="-3.9" upper="1.5" velocity="1.0"/>
   </joint>
@@ -707,10 +729,10 @@
         value="0.0701242408063442" />
       <inertia
-        ixx="1.73265934767466E-05"
-        ixy="2.38363792824069E-07"
-        ixz="7.96430204321056E-08"
-        iyy="4.11044416077217E-05"
-        iyz="-9.41955638215997E-07"
-        izz="2.38851808140542E-05" />
+        ixx="0.001"
+        ixy="0"
+        ixz="0"
+        iyy="0.001"
+        iyz="0"
+        izz="0.001" />
     </inertial>
     <visual>
@@ -750,6 +772,5 @@
     <axis
       xyz="0 0 1" />
-    <!-- unconstrained range for now -->
     <limit effort="100" lower="-1.53" upper="0.79" velocity="1.0"/>
-  </joint>
+  </joint> -->
 </robot>

Commit message: Base working, arm next

File: stretch_description/urdf/stretch_main.xacro (robot description, xacro)
@@ -134,5 +134,5 @@
     <axis xyz="0 0 1" />
   </joint>
-  <link name="caster_link">
+  <link name="link_caster">
     <collision>
       <geometry>
@@ -177,7 +177,7 @@
     </inertial>
   </link>
-  <joint name="caster_joint" type="fixed">
+  <joint name="joint_caster" type="fixed">
     <parent link="base_link"/>
-    <child link="caster_link"/>
+    <child link="link_caster"/>
     <origin xyz="-0.245 0.0 0.032" rpy="${-M_PI/2} 0 0"/>
     <axis xyz="0 0 1" />
@@ -236,5 +236,5 @@
       xyz="0 0 0" />
   </joint>
-  <!-- <link
+  <link
     name="link_lift">
     <inertial>
@@ -773,4 +773,4 @@
       xyz="0 0 1" />
     <limit effort="100" lower="-1.53" upper="0.79" velocity="1.0"/>
-  </joint> -->
+  </joint>
 </robot>

File: stretch_gazebo/urdf/stretch_gazebo.urdf.xacro (robot description, xacro)
@@ -71,3 +71,13 @@
       <material>Gazebo/Gray</material>
   </gazebo>
+    <plugin
+      filename="libignition-gazebo-diff-drive-system.so"
+      name="ignition::gazebo::systems::DiffDrive">
+      <left_joint>joint_left_wheel</left_joint>
+      <right_joint>joint_right_wheel</right_joint>
+      <wheel_separation>0.315</wheel_separation>
+      <wheel_radius>0.05</wheel_radius>
+      <odom_publish_frequency>1</odom_publish_frequency>
+      <topic>cmd_vel</topic>
+  </plugin>
 </robot>
