Commit message: Gripper stuff

File: stretch_description/urdf/stretch_gripper.xacro (robot description, xacro)
@@ -109,5 +109,5 @@
     <axis
       xyz="0 0 1" />
-    <limit effort="100" lower="-0.6" upper="0.6" velocity="1.0"/>
+    <limit effort="100" lower="-0.5" upper="0.25" velocity="1.0"/>
   </joint>
   <link
@@ -216,5 +216,5 @@
     <axis
       xyz="0 0 1" />
-    <limit effort="100" lower="-0.6" upper="0.6" velocity="1.0"/>
+    <limit effort="100" lower="-0.5" upper="0.25" velocity="1.0"/>
   </joint>
   <link

Commit message: FollowJointTrajectory advanced implementation

File: stretch_description/urdf/stretch_gripper.xacro (robot description, xacro)
@@ -109,5 +109,5 @@
     <axis
       xyz="0 0 1" />
-    <limit effort="100" lower="-0.6" upper="0.6" velocity="1.0"/>
+    <limit effort="100" lower="-0.526" upper="0.263" velocity="1.0"/>
   </joint>
   <link
@@ -216,5 +216,5 @@
     <axis
       xyz="0 0 1" />
-    <limit effort="100" lower="-0.6" upper="0.6" velocity="1.0"/>
+    <limit effort="100" lower="-0.526" upper="0.263" velocity="1.0"/>
   </joint>
   <link
