Commit message: New dae files and port to xacro

File: stretch_description/urdf/stretch_aruco.xacro (robot description, xacro)
@@ -114,5 +114,5 @@
         rpy="0 0 0" />
       <mass
-        value="0.000399141592653546" />
+        value="0.0000399141592653546" />
       <inertia
         ixx="0"
@@ -167,5 +167,5 @@
         rpy="0 0 0" />
       <mass
-        value="0.000224999999999975" />
+        value="0.00000224999999999975" />
       <inertia
         ixx="0"
@@ -220,5 +220,5 @@
         rpy="0 0 0" />
       <mass
-        value="0.000225" />
+        value="0.00000225" />
       <inertia
         ixx="0"

File: stretch_description/urdf/stretch_description.xacro (robot description, xacro)
@@ -1,5 +1,5 @@
 <?xml version="1.0"?>
 <robot xmlns:xacro="http://www.ros.org/wiki/xacro" name="stretch_description">
-  <!-- <xacro:include filename="stretch_gripper.xacro" /> -->
+  <xacro:include filename="stretch_gripper.xacro" />
   <!--<xacro:include filename="stretch_gripper_with_puller.xacro" />-->
   <!--<xacro:include filename="stretch_dry_erase_marker.xacro" />-->

File: stretch_description/urdf/stretch_gripper.xacro (robot description, xacro)
@@ -2,6 +2,6 @@
 <robot xmlns:xacro="http://www.ros.org/wiki/xacro" name="stretch_gripper">
   <xacro:property name="scale_finger_length" value="0.9" />
-  <xacro:property name="gripper_joint_damping" value="21.75"/>
-  <xacro:property name="gripper_joint_friction" value="3.48"/>
+  <xacro:property name="gripper_joint_damping" value="0.75"/>
+  <xacro:property name="gripper_joint_friction" value="2.48"/>
   <xacro:property name="gripper_joint_spring_stiffness" value="0"/>
   <xacro:property name="gripper_joint_spring_reference" value="0"/>
@@ -13,5 +13,5 @@
         rpy="0 0 0" />
       <mass
-        value="0.101902711393094" />
+        value="0.000101902711393094" />
       <inertia
         ixx="0.001"
@@ -28,11 +28,6 @@
       <geometry>
         <mesh
-          filename="package://stretch_description/meshes/link_gripper.STL" />
-      </geometry>
-      <material
-        name="">
-        <color
-          rgba="0.792156862745098 0.819607843137255 0.933333333333333 1" />
-      </material>
+          filename="package://stretch_description/meshes/link_gripper.dae" />
+      </geometry>
     </visual>
     <collision>
@@ -66,5 +61,5 @@
         rpy="0 0 0" />
       <mass
-        value="0.0476207785199474" />
+        value="0.000476207785199474" />
       <inertia
         ixx="0.001"
@@ -81,11 +76,6 @@
       <geometry>
         <mesh
-          filename="package://stretch_description/meshes/link_gripper_finger_left.STL" scale="${scale_finger_length} 1.0 1.0"/>
-      </geometry>
-      <material
-        name="">
-        <color
-          rgba="0.792156862745098 0.819607843137255 0.933333333333333 1" />
-      </material>
+          filename="package://stretch_description/meshes/link_gripper_finger_left.dae" scale="${scale_finger_length} 1.0 1.0"/>
+      </geometry>
     </visual>
     <collision>
@@ -121,5 +111,5 @@
         rpy="0 0 0" />
       <mass
-        value="0.00382159917455729" />
+        value="0.000382159917455729" />
         <inertia
         ixx="0.001"
@@ -136,11 +126,6 @@
       <geometry>
         <mesh
-          filename="package://stretch_description/meshes/link_gripper_fingertip_left.STL" />
-      </geometry>
-      <material
-        name="">
-        <color
-          rgba="0.250980392156863 0.250980392156863 0.250980392156863 1" />
-      </material>
+          filename="package://stretch_description/meshes/link_gripper_fingertip_left.dae" />
+      </geometry>
     </visual>
     <collision>
@@ -174,5 +159,5 @@
         rpy="0 0 0" />
       <mass
-        value="0.0476207785199481" />
+        value="0.000476207785199481" />
         <inertia
         ixx="0.001"
@@ -189,11 +174,6 @@
       <geometry>
         <mesh
-          filename="package://stretch_description/meshes/link_gripper_finger_right.STL" scale="${scale_finger_length} 1.0 1.0"/>
-      </geometry>
-      <material
-        name="">
-        <color
-          rgba="0.792156862745098 0.819607843137255 0.933333333333333 1" />
-      </material>
+          filename="package://stretch_description/meshes/link_gripper_finger_right.dae" scale="${scale_finger_length} 1.0 1.0"/>
+      </geometry>
     </visual>
     <collision>
@@ -229,5 +209,5 @@
         rpy="0 0 0" />
       <mass
-        value="0.00382160037319545" />
+        value="0.000382160037319545" />
       <inertia
         ixx="0.001"
@@ -244,11 +224,6 @@
       <geometry>
         <mesh
-          filename="package://stretch_description/meshes/link_gripper_fingertip_right.STL" />
-      </geometry>
-      <material
-        name="">
-        <color
-          rgba="0.250980392156863 0.250980392156863 0.250980392156863 1" />
-      </material>
+          filename="package://stretch_description/meshes/link_gripper_fingertip_right.dae" />
+      </geometry>
     </visual>
     <collision>

File: stretch_description/urdf/stretch_laser_range_finder.xacro (robot description, xacro)
@@ -23,11 +23,6 @@
       <geometry>
         <mesh
-          filename="package://stretch_description/meshes/laser.STL" />
+          filename="package://stretch_description/meshes/laser.dae" />
       </geometry>
-      <material
-        name="">
-        <color
-          rgba="0.250980392156863 0.250980392156863 0.250980392156863 1" />
-      </material>
     </visual>
     <collision>

File: stretch_description/urdf/stretch_main.xacro (robot description, xacro)
@@ -2,8 +2,12 @@
 <robot xmlns:xacro="http://www.ros.org/wiki/xacro" name="stretch_main">
   <xacro:property name="M_PI" value="3.1415926535897931" />
-  <xacro:property name="joint_damping" value="21.75"/>
-  <xacro:property name="joint_friction" value="3.48"/>
+  <xacro:property name="joint_damping" value="0.75"/>
+  <xacro:property name="joint_friction" value="2.48"/>
   <xacro:property name="joint_spring_stiffness" value="0"/>
   <xacro:property name="joint_spring_reference" value="0"/>
+  <xacro:property name="caster_damping" value="0.005"/>
+  <xacro:property name="caster_friction" value="0.001"/>
+  <xacro:property name="caster_velocity_limit" value="5.0"/>
+  <xacro:property name="caster_effort_limit" value="100"/>
   <link
     name="base_link">
@@ -28,20 +32,15 @@
       <geometry>
         <mesh
+          filename="package://stretch_description/meshes/base_link.dae" />
+      </geometry>
+    </visual>
+    <collision>
+      <origin
+        xyz="0 0 0"
+        rpy="0 0 0" />
+      <geometry>
+        <mesh
           filename="package://stretch_description/meshes/base_link.STL" />
       </geometry>
-      <material
-        name="">
-        <color
-          rgba="0.792156862745098 0.819607843137255 0.933333333333333 1" />
-      </material>
-    </visual>
-    <collision>
-      <origin
-        xyz="0 0 0"
-        rpy="0 0 0" />
-      <geometry>
-        <mesh
-          filename="package://stretch_description/meshes/base_link.STL" />
-      </geometry>
     </collision>
   </link>
@@ -68,11 +67,6 @@
       <geometry>
         <mesh
-          filename="package://stretch_description/meshes/link_right_wheel.STL" />
-      </geometry>
-      <material
-        name="">
-        <color
-          rgba="0.792156862745098 0.819607843137255 0.933333333333333 1" />
-      </material>
+          filename="package://stretch_description/meshes/link_right_wheel.dae" />
+      </geometry>
     </visual>
     <collision>
@@ -122,11 +116,6 @@
       <geometry>
         <mesh
-          filename="package://stretch_description/meshes/link_left_wheel.STL" />
-      </geometry>
-      <material
-        name="">
-        <color
-          rgba="0.792156862745098 0.819607843137255 0.933333333333333 1" />
-      </material>
+          filename="package://stretch_description/meshes/link_left_wheel.dae" />
+      </geometry>
     </visual>
     <collision>
@@ -153,5 +142,47 @@
       xyz="0 0 1" />
       <dynamics damping="${joint_damping}" friction="${joint_friction}" spring_reference="${joint_spring_reference}" spring_stiffness="{joint_spring_stiffness}"/>
-  </joint>
+      <!-- <dynamics damping="21.75" friction="3.48" spring_reference="0.0" spring_stiffness="0.0"/> -->
+  </joint>
+  <!-- Representing a ball joint -->
+  <joint name="caster_joint_theta" type="continuous">
+    <origin xyz="-0.245 0.0 0.032" rpy="${-M_PI/2} 0 0"/>
+    <parent link="base_link"/>
+    <child link="caster_link_theta"/>
+    <axis xyz="0 1 0" />
+    <dynamics friction="${caster_friction}" damping="${caster_damping}" />
+    <limit lower="${-pi/2}" upper="${-pi/2}" velocity="${caster_velocity_limit}" effort="${caster_effort_limit}" />
+  </joint>
+  <link name="caster_link_theta">
+    <inertial>
+      <mass value="0.0025" />
+      <inertia ixx="5.8083e-4" ixy="0" ixz="0" iyy="3.0833e-5" iyz="0" izz="5.9083e-4" />
+    </inertial>
+  </link>
+  <joint name="caster_joint_psi" type="continuous">
+    <parent link="caster_link_theta"/>
+    <child link="caster_link_psi"/>
+    <axis xyz="0 0 1" />
+    <dynamics friction="${caster_friction}" damping="${caster_damping}" />
+    <limit lower="${-pi/2}" upper="${-pi/2}" velocity="${caster_velocity_limit}" effort="${caster_effort_limit}" />
+  </joint>
+  <link name="caster_link_psi">
+    <inertial>
+      <mass value="0.0025" />
+      <inertia ixx="5.8083e-4" ixy="0" ixz="0" iyy="3.0833e-5" iyz="0" izz="5.9083e-4" />
+    </inertial>
+  </link>
+  <joint name="caster_joint_phi" type="continuous">
+    <parent link="caster_link_theta"/>
+    <child link="caster_link_phi"/>
+    <axis xyz="1 0 0" />
+    <dynamics friction="${caster_friction}" damping="${caster_damping}" />
+  </joint>
+  <link name="caster_link_phi">
+    <inertial>
+      <mass value="0.0025" />
+      <inertia ixx="5.8083e-4" ixy="0" ixz="0" iyy="3.0833e-5" iyz="0" izz="5.9083e-4" />
+      <limit lower="${-pi/2}" upper="${-pi/2}" velocity="${caster_velocity_limit}" effort="${caster_effort_limit}" />
+    </inertial>
+  </link>
   <link name="link_caster">
     <collision>
@@ -169,4 +200,13 @@
           </ode>
         </friction>
+        <contact>
+          <ode>
+            <soft_cfm>0</soft_cfm>
+            <soft_erp>0.2</soft_erp>
+            <kp>1e+13</kp>
+            <kd>1</kd>
+            <min_depth>0.001</min_depth>
+          </ode>
+        </contact>
       </surface>
     </collision>
@@ -177,11 +217,6 @@
       <geometry>
         <mesh
-          filename="package://stretch_description/meshes/omni_wheel_m.STL" />
-      </geometry>
-      <material
-        name="">
-        <color
-          rgba="0.792156862745098 0.819607843137255 0.933333333333333 1" />
-      </material>
+          filename="package://stretch_description/meshes/omni_wheel_m.dae" />
+      </geometry>
     </visual>
     <inertial>
@@ -198,8 +233,8 @@
   </link>
   <joint name="joint_caster" type="fixed">
-    <parent link="base_link"/>
+    <parent link="caster_link_phi"/>
+    <!-- <parent link="base_link"/> -->
     <child link="link_caster"/>
-    <origin xyz="-0.245 0.0 0.032" rpy="${-M_PI/2} 0 0"/>
-    <axis xyz="0 0 1" />
+    <!-- <origin xyz="-0.245 0.0 0.032" rpy="${-M_PI/2} 0 0"/> -->
   </joint>
   <link
@@ -207,29 +242,24 @@
     <inertial>
       <origin
-        xyz="0.00755818572975822 0.773971284176834 0.00647313086620024"
-        rpy="0 0 0" />
-      <mass
-        value="0.749143203376401" />
-      <inertia
-        ixx="0.0709854511954588"
-        ixy="-0.00433428742758457"
-        ixz="-0.000186110788697573"
-        iyy="0.000437922053342648"
-        iyz="-0.00288788257713431"
-        izz="0.071104808501661" />
-    </inertial>
-    <visual>
-      <origin
-        xyz="0 0 0"
-        rpy="0 0 0" />
-      <geometry>
-        <mesh
-          filename="package://stretch_description/meshes/link_mast.STL" />
-      </geometry>
-      <material
-        name="">
-        <color
-          rgba="0.792156862745098 0.819607843137255 0.933333333333333 1" />
-      </material>
+        xyz="-0.109461304328163 -0.000741018909047708 0.0914915269429946"
+        rpy="0 0 0" />
+      <mass
+        value="0.05" />
+      <inertia
+        ixx="0.001"
+        ixy="0.0"
+        ixz="0.0"
+        iyy="0.001"
+        iyz="0.0"
+        izz="0.001" />
+    </inertial>
+    <visual>
+      <origin
+        xyz="0 0 0"
+        rpy="0 0 0" />
+      <geometry>
+        <mesh
+          filename="package://stretch_description/meshes/link_mast.dae" />
+      </geometry>
     </visual>
     <collision>
@@ -263,26 +293,21 @@
         rpy="0 0 0" />
       <mass
-        value="0.444820831236007" />
-      <inertia
-        ixx="0.000567192946271367"
-        ixy="-0.00024607534789508"
-        ixz="-0.000128108442260574"
-        iyy="0.00127108364478659"
-        iyz="7.61916855070339E-06"
-        izz="0.00137296635099006" />
-    </inertial>
-    <visual>
-      <origin
-        xyz="0 0 0"
-        rpy="0 0 0" />
-      <geometry>
-        <mesh
-          filename="package://stretch_description/meshes/link_lift.STL" />
-      </geometry>
-      <material
-        name="">
-        <color
-          rgba="0.792156862745098 0.819607843137255 0.933333333333333 1" />
-      </material>
+        value="0.044820831236007" />
+      <inertia
+        ixx="0.001"
+        ixy="0.0"
+        ixz="0.0"
+        iyy="0.001"
+        iyz="0.0"
+        izz="0.001" />
+    </inertial>
+    <visual>
+      <origin
+        xyz="0 0 0"
+        rpy="0 0 0" />
+      <geometry>
+        <mesh
+          filename="package://stretch_description/meshes/link_lift.dae" />
+      </geometry>
     </visual>
     <collision>
@@ -308,9 +333,7 @@
     <axis
   xyz="0 0 1" />
-    <!-- for now: hand copied range_m: from lift: from ~/repos/stretch_fleet/stretch-re1-1001/stretch_re1_factory_params.yaml -->
-    <!--<limit effort="100" lower="0.0" upper="1.095" velocity="1.0"/>-->
-    <!-- copied value did not reach the top of mesh model with GUI sliders and RViz -->
     <limit effort="100" lower="-0.1033" upper="0.9967" velocity="1.0"/>
-    <dynamics damping="${joint_damping}" friction="${joint_friction}" spring_reference="${joint_spring_reference}" spring_stiffness="{joint_spring_stiffness}"/>
+    <!-- Make this high friction so gripper does not fall -->
+    <dynamics damping="10" friction="10.48" spring_reference="${joint_spring_reference}" spring_stiffness="{joint_spring_stiffness}"/>
   </joint>
   <link
@@ -321,26 +344,21 @@
         rpy="0 0 0" />
       <mass
-        value="0.0676525455789735" />
-      <inertia
-        ixx="0.001"
-        ixy="0"
-        ixz="0"
-        iyy="0.001"
-        iyz="0"
-        izz="0.001" />
-    </inertial>
-    <visual>
-      <origin
-        xyz="0 0 0"
-        rpy="0 0 0" />
-      <geometry>
-        <mesh
-          filename="package://stretch_description/meshes/link_arm_l4.STL" />
-      </geometry>
-      <material
-        name="">
-        <color
-          rgba="0.792156862745098 0.819607843137255 0.933333333333333 1" />
-      </material>
+        value="0.00676525455789735" />
+      <inertia
+        ixx="0.001"
+        ixy="0"
+        ixz="0"
+        iyy="0.001"
+        iyz="0"
+        izz="0.001" />
+    </inertial>
+    <visual>
+      <origin
+        xyz="0 0 0"
+        rpy="0 0 0" />
+      <geometry>
+        <mesh
+          filename="package://stretch_description/meshes/link_arm_l4.dae" />
+      </geometry>
     </visual>
     <collision>
@@ -374,26 +392,21 @@
         rpy="0 0 0" />
       <mass
-        value="0.0626921047058405" />
-      <inertia
-        ixx="0.001"
-        ixy="0"
-        ixz="0"
-        iyy="0.001"
-        iyz="0"
-        izz="0.001" />
-    </inertial>
-    <visual>
-      <origin
-        xyz="0 0 0"
-        rpy="0 0 0" />
-      <geometry>
-        <mesh
-          filename="package://stretch_description/meshes/link_arm_l3.STL" />
-      </geometry>
-      <material
-        name="">
-        <color
-          rgba="0.792156862745098 0.819607843137255 0.933333333333333 1" />
-      </material>
+        value="0.00626921047058405" />
+      <inertia
+        ixx="0.001"
+        ixy="0"
+        ixz="0"
+        iyy="0.001"
+        iyz="0"
+        izz="0.001" />
+    </inertial>
+    <visual>
+      <origin
+        xyz="0 0 0"
+        rpy="0 0 0" />
+      <geometry>
+        <mesh
+          filename="package://stretch_description/meshes/link_arm_l3.dae" />
+      </geometry>
     </visual>
     <collision>
@@ -419,5 +432,4 @@
     <axis
   xyz="0 0 1" />
-    <!-- 0.13 = 0.52/4-->
     <limit effort="100" lower="0.0" upper="0.13" velocity="1.0"/>
     <dynamics damping="${joint_damping}" friction="${joint_friction}" spring_reference="${joint_spring_reference}" spring_stiffness="{joint_spring_stiffness}"/>
@@ -430,26 +442,21 @@
         rpy="0 0 0" />
       <mass
-        value="0.0569074368576238" />
-      <inertia
-        ixx="0.001"
-        ixy="0"
-        ixz="0"
-        iyy="0.001"
-        iyz="0"
-        izz="0.001" />
-    </inertial>
-    <visual>
-      <origin
-        xyz="0 0 0"
-        rpy="0 0 0" />
-      <geometry>
-        <mesh
-          filename="package://stretch_description/meshes/link_arm_l2.STL" />
-      </geometry>
-      <material
-        name="">
-        <color
-          rgba="0.792156862745098 0.819607843137255 0.933333333333333 1" />
-      </material>
+        value="0.00569074368576238" />
+      <inertia
+        ixx="0.001"
+        ixy="0"
+        ixz="0"
+        iyy="0.001"
+        iyz="0"
+        izz="0.001" />
+    </inertial>
+    <visual>
+      <origin
+        xyz="0 0 0"
+        rpy="0 0 0" />
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
File: stretch_description/urdf/stretch_respeaker.xacro (robot description, xacro)
@@ -7,5 +7,5 @@
         rpy="0 0 0" />
       <mass
-        value="0.00969129410417277" />
+        value="0.0000969129410417277" />
       <inertia
         ixx="8.95656300428405E-07"
