Commit message: Gripper, lidar

File: stretch_description/urdf/stretch_description.xacro (robot description, xacro)
@@ -5,7 +5,7 @@
   <!--<xacro:include filename="stretch_dry_erase_marker.xacro" />-->
   <xacro:include filename="stretch_main.xacro" />
-  <!-- <xacro:include filename="stretch_aruco.xacro" />
-  <xacro:include filename="stretch_d435i.xacro" />
+  <!-- <xacro:include filename="stretch_aruco.xacro" /> -->
+  <!-- <xacro:include filename="stretch_d435i.xacro" /> -->
   <xacro:include filename="stretch_laser_range_finder.xacro" />
-  <xacro:include filename="stretch_respeaker.xacro" /> -->
+  <!-- <xacro:include filename="stretch_respeaker.xacro" /> -->
 </robot>

File: stretch_description/urdf/stretch_main.xacro (robot description, xacro)
@@ -279,6 +279,7 @@
     name="joint_lift"
     type="prismatic">
-    <origin
-      xyz="-0.0369217062323472 0.165471199999996 -0.000341653286793524"
+    <!-- Y: 0.165471199999996 -->
+    <origin
+      xyz="-0.0369217062323472 0.2687712 -0.000341653286793524"
       rpy="-1.57079632679552 1.5615431375292 -6.2942004366467E-13" />
     <parent
@@ -288,5 +289,6 @@
     <axis
 	xyz="0 0 1" />
-  <limit effort="100" lower="0.0" upper="1.1" velocity="1.0"/>
+  <!-- <limit effort="100" lower="0.0" upper="1.1" velocity="1.0"/> -->
+  <limit effort="100" lower="-0.1033" upper="0.9967" velocity="1.0"/>
   </joint>
   <link

Commit message: Temp push for moveit2 integration

File: stretch_description/urdf/stretch_description.xacro (robot description, xacro)
@@ -5,7 +5,7 @@
   <!--<xacro:include filename="stretch_dry_erase_marker.xacro" />-->
   <xacro:include filename="stretch_main.xacro" />
-  <!-- <xacro:include filename="stretch_aruco.xacro" /> -->
+  <xacro:include filename="stretch_aruco.xacro" />
   <!-- <xacro:include filename="stretch_d435i.xacro" /> -->
   <xacro:include filename="stretch_laser_range_finder.xacro" />
-  <!-- <xacro:include filename="stretch_respeaker.xacro" /> -->
+  <xacro:include filename="stretch_respeaker.xacro" />
 </robot>

File: stretch_description/urdf/stretch_test.urdf (robot description, URDF)
Before this commit: robot stretch_main, 16 links, 15 joints
Links:
- added link link_aruco_inner_wrist, mass 0.000225; collision mesh filename=package://stretch_description/meshes/link_aruco_inner_wrist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; visual mesh filename=package://stretch_description/meshes/link_aruco_inner_wrist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
- added link link_aruco_left_base, mass 3.59999999990368E-06; collision mesh filename=package://stretch_description/meshes/link_aruco_left_base.S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; visual mesh filename=package://stretch_description/meshes/link_aruco_left_base.S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
- added link link_aruco_right_base, mass 3.59999999990368E-06; collision mesh filename=package://stretch_description/meshes/link_aruco_right_base.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; visual mesh filename=package://stretch_description/meshes/link_aruco_right_base.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
- added link link_aruco_shoulder, mass 0.000399141592653546; collision mesh filename=package://stretch_description/meshes/link_aruco_shoulder.STL; visual mesh filename=package://stretch_description/meshes/link_aruco_shoulder.STL
- added link link_aruco_top_wrist, mass 0.000224999999999975; collision mesh filename=package://stretch_description/meshes/link_aruco_top_wrist.S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; visual mesh filename=package://stretch_description/meshes/link_aruco_top_wrist.S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
- added link respeaker_base, mass 0.00969129410417277; collision mesh filename=package://stretch_description/meshes/link_respeaker.STL; visual mesh filename=package://stretch_description/meshes/link_respeaker.STL
Joints:
- added joint joint_aruco_inner_wrist: type fixed, parent link_arm_l0, child link_aruco_inner_wrist, origin xyz=0.0472499999999947 -0.0119000000000034 -0.0272499999991938 rpy=3.14159265358979 4.23377442363088E-14 3.14159265358979, axis 0 0 0
- added joint joint_aruco_left_base: type fixed, parent base_link, child link_aruco_left_base, origin xyz=-0.00500000000000014 0.1304972 0.1597482 rpy=0 0 -1.5707963267949, axis 0 0 0
- added joint joint_aruco_right_base: type fixed, parent base_link, child link_aruco_right_base, origin xyz=-0.00500000000000014 -0.1304972 0.1597482 rpy=0 0 -1.5707963267949, axis 0 0 0
- added joint joint_aruco_shoulder: type fixed, parent link_lift, child link_aruco_shoulder, origin xyz=-0.0133768876375287 0.0558540528812078 0.0861368272417975 rpy=-1.53998860117704E-29 3.55962409571165E-15 0.0, axis 0 0 0
- added joint joint_aruco_top_wrist: type fixed, parent link_arm_l0, child link_aruco_top_wrist, origin xyz=0.0472500000000019 0.0292850000000015 0 rpy=1.5707963267949 -8.03728587323464E-15 3.14159265358979, axis 0 0 0
- added joint joint_respeaker: type fixed, parent link_mast, child respeaker_base, origin xyz=1.09074743137871E-05 1.36992 0.00303572796911382 rpy=1.57079632679553 0.0 3.14159265358916, axis 0 0 0

Commit message: Arm, head and gripper

File: stretch_description/urdf/stretch_description.xacro (robot description, xacro)
@@ -6,5 +6,5 @@
   <xacro:include filename="stretch_main.xacro" />
   <xacro:include filename="stretch_aruco.xacro" />
-  <xacro:include filename="stretch_d435i.xacro" />
+  <!-- <xacro:include filename="stretch_d435i.xacro" /> -->
   <xacro:include filename="stretch_laser_range_finder.xacro" />
   <xacro:include filename="stretch_respeaker.xacro" />

File: stretch_description/urdf/stretch_main.xacro (robot description, xacro)
@@ -1,4 +1,5 @@
 <?xml version="1.0"?>
 <robot xmlns:xacro="http://www.ros.org/wiki/xacro" name="stretch_main">
+  <xacro:property name="M_PI" value="3.1415926535897931" />
   <link
     name="base_link">
@@ -147,4 +148,53 @@
       xyz="0 0 1" />
   </joint>
+  <link name="link_caster">
+    <collision>
+      <geometry>
+        <sphere radius="0.032"/>
+      </geometry>
+      <origin rpy="0 0 0" xyz="0 0 0"/>
+      <surface>
+        <friction>
+          <ode>
+            <mu>0</mu>
+            <mu2>0</mu2>
+            <slip1>1.0</slip1>
+            <slip2>1.0</slip2>
+          </ode>
+        </friction>
+      </surface>
+    </collision>
+    <visual>
+      <origin
+        xyz="0 0 0"
+        rpy="0 0 0" />
+      <geometry>
+        <mesh
+          filename="package://stretch_description/meshes/omni_wheel_m.STL" />
+      </geometry>
+      <material
+        name="">
+        <color
+          rgba="0.792156862745098 0.819607843137255 0.933333333333333 1" />
+      </material>
+    </visual>
+    <inertial>
+      <mass value="0.01" />
+      <origin xyz="0 0 0" />
+      <inertia
+        ixx="0.001"
+        ixy="0"
+        ixz="0"
+        iyy="0.001"
+        iyz="0"
+        izz="0.001" />
+    </inertial>
+  </link>
+  <joint name="joint_caster" type="fixed">
+    <parent link="base_link"/>
+    <child link="link_caster"/>
+    <origin xyz="-0.245 0.0 0.032" rpy="${-M_PI/2} 0 0"/>
+    <axis xyz="0 0 1" />
+  </joint>
   <link
     name="link_mast">
@@ -244,5 +294,5 @@
     type="prismatic">
     <origin
-      xyz="-0.0369217062323472 0.165471199999996 -0.000341653286793524"
+      xyz="-0.0369217062323472 0.266771199999996 -0.000341653286793524"
       rpy="-1.57079632679552 1.5615431375292 -6.2942004366467E-13" />
     <parent
@@ -255,5 +305,5 @@
   <!--<limit effort="100" lower="0.0" upper="1.095" velocity="1.0"/>-->
   <!-- copied value did not reach the top of mesh model with GUI sliders and RViz -->
-  <limit effort="100" lower="0.0" upper="1.1" velocity="1.0"/>
+  <limit effort="100" lower="-0.1033" upper="0.9967" velocity="1.0"/>
   </joint>
   <link

Commit message: Add xacro spawn and port sensors

File: stretch_description/urdf/stretch_description.xacro (robot description, xacro)
@@ -1,5 +1,5 @@
 <?xml version="1.0"?>
 <robot xmlns:xacro="http://www.ros.org/wiki/xacro" name="stretch_description">
-  <xacro:include filename="stretch_gripper.xacro" />
+  <!-- <xacro:include filename="stretch_gripper.xacro" /> -->
   <!--<xacro:include filename="stretch_gripper_with_puller.xacro" />-->
   <!--<xacro:include filename="stretch_dry_erase_marker.xacro" />-->

File: stretch_description/urdf/stretch_gripper.xacro (robot description, xacro)
@@ -2,4 +2,8 @@
 <robot xmlns:xacro="http://www.ros.org/wiki/xacro" name="stretch_gripper">
   <xacro:property name="scale_finger_length" value="0.9" />
+  <xacro:property name="gripper_joint_damping" value="21.75"/>
+  <xacro:property name="gripper_joint_friction" value="3.48"/>
+  <xacro:property name="gripper_joint_spring_stiffness" value="0"/>
+  <xacro:property name="gripper_joint_spring_reference" value="0"/>
   <link
     name="link_gripper">
@@ -11,10 +15,10 @@
         value="0.101902711393094" />
       <inertia
-        ixx="2.79241618017607E-05"
-        ixy="-1.10819247449605E-05"
-        ixz="-1.50343284036654E-05"
-        iyy="3.67945130513069E-05"
-        iyz="-4.33280448535579E-06"
-        izz="4.14524691955231E-05" />
+        ixx="0.001"
+        ixy="0"
+        ixz="0"
+        iyy="0.001"
+        iyz="0"
+        izz="0.001" />
     </inertial>
     <visual>
@@ -42,6 +46,4 @@
     </collision>
   </link>
-  <!-- rpy="3.1416 0 1.5708" -->
-  <!-- rpy="0.0 0 1.5708" -->
   <joint
     name="joint_gripper"
@@ -66,10 +68,10 @@
         value="0.0476207785199474" />
       <inertia
-        ixx="0"
-        ixy="0"
-        ixz="0"
-        iyy="0"
-        iyz="0"
-        izz="0" />
+        ixx="0.001"
+        ixy="0"
+        ixz="0"
+        iyy="0.001"
+        iyz="0"
+        izz="0.001" />
     </inertial>
     <visual>
@@ -110,4 +112,5 @@
       xyz="0 0 1" />
     <limit effort="100" lower="-0.6" upper="0.6" velocity="1.0"/>
+    <dynamics damping="${gripper_joint_damping}" friction="${gripper_joint_friction}" spring_reference="${gripper_joint_spring_reference}" spring_stiffness="{gripper_joint_spring_stiffness}"/>
   </joint>
   <link
@@ -119,11 +122,11 @@
       <mass
         value="0.00382159917455729" />
-      <inertia
-        ixx="0"
-        ixy="0"
-        ixz="0"
-        iyy="0"
-        iyz="0"
-        izz="0" />
+        <inertia
+        ixx="0.001"
+        ixy="0"
+        ixz="0"
+        iyy="0.001"
+        iyz="0"
+        izz="0.001" />
     </inertial>
     <visual>
@@ -172,11 +175,11 @@
       <mass
         value="0.0476207785199481" />
-      <inertia
-        ixx="0"
-        ixy="0"
-        ixz="0"
-        iyy="0"
-        iyz="0"
-        izz="0" />
+        <inertia
+        ixx="0.001"
+        ixy="0"
+        ixz="0"
+        iyy="0.001"
+        iyz="0"
+        izz="0.001" />
     </inertial>
     <visual>
@@ -217,4 +220,5 @@
       xyz="0 0 1" />
     <limit effort="100" lower="-0.6" upper="0.6" velocity="1.0"/>
+    <dynamics damping="${gripper_joint_damping}" friction="${gripper_joint_friction}" spring_reference="${gripper_joint_spring_reference}" spring_stiffness="{gripper_joint_spring_stiffness}"/>
   </joint>
   <link
@@ -227,10 +231,10 @@
         value="0.00382160037319545" />
       <inertia
-        ixx="0"
-        ixy="0"
-        ixz="0"
-        iyy="0"
-        iyz="0"
-        izz="0" />
+        ixx="0.001"
+        ixy="0"
+        ixz="0"
+        iyy="0.001"
+        iyz="0"
+        izz="0.001" />
     </inertial>
     <visual>

File: stretch_description/urdf/stretch_main.xacro (robot description, xacro)
@@ -2,4 +2,8 @@
 <robot xmlns:xacro="http://www.ros.org/wiki/xacro" name="stretch_main">
   <xacro:property name="M_PI" value="3.1415926535897931" />
+  <xacro:property name="joint_damping" value="21.75"/>
+  <xacro:property name="joint_friction" value="3.48"/>
+  <xacro:property name="joint_spring_stiffness" value="0"/>
+  <xacro:property name="joint_spring_reference" value="0"/>
   <link
     name="base_link">
@@ -51,10 +55,10 @@
         value="0.00356714564938475" />
       <inertia
-        ixx="0"
-        ixy="0"
-        ixz="0"
-        iyy="0"
-        iyz="0"
-        izz="0" />
+        ixx="0.001"
+        ixy="0"
+        ixz="0"
+        iyy="0.001"
+        iyz="0"
+        izz="0.001" />
     </inertial>
     <visual>
@@ -94,4 +98,5 @@
     <axis
       xyz="0 0 1" />
+      <dynamics damping="${joint_damping}" friction="${joint_friction}" spring_reference="${joint_spring_reference}" spring_stiffness="{joint_spring_stiffness}"/>
   </joint>
   <link
@@ -104,10 +109,10 @@
         value="0.00356714564938459" />
       <inertia
-        ixx="0"
-        ixy="0"
-        ixz="0"
-        iyy="0"
-        iyz="0"
-        izz="0" />
+        ixx="0.001"
+        ixy="0"
+        ixz="0"
+        iyy="0.001"
+        iyz="0"
+        izz="0.001" />
     </inertial>
     <visual>
@@ -147,4 +152,5 @@
     <axis
       xyz="0 0 1" />
+      <dynamics damping="${joint_damping}" friction="${joint_friction}" spring_reference="${joint_spring_reference}" spring_stiffness="{joint_spring_stiffness}"/>
   </joint>
   <link name="link_caster">
@@ -301,9 +307,10 @@
       link="link_lift" />
     <axis
-	xyz="0 0 1" />
-  <!-- for now: hand copied range_m: from lift: from ~/repos/stretch_fleet/stretch-re1-1001/stretch_re1_factory_params.yaml -->
-  <!--<limit effort="100" lower="0.0" upper="1.095" velocity="1.0"/>-->
-  <!-- copied value did not reach the top of mesh model with GUI sliders and RViz -->
-  <limit effort="100" lower="-0.1033" upper="0.9967" velocity="1.0"/>
+  xyz="0 0 1" />
+    <!-- for now: hand copied range_m: from lift: from ~/repos/stretch_fleet/stretch-re1-1001/stretch_re1_factory_params.yaml -->
+    <!--<limit effort="100" lower="0.0" upper="1.095" velocity="1.0"/>-->
+    <!-- copied value did not reach the top of mesh model with GUI sliders and RViz -->
+    <limit effort="100" lower="-0.1033" upper="0.9967" velocity="1.0"/>
+    <dynamics damping="${joint_damping}" friction="${joint_friction}" spring_reference="${joint_spring_reference}" spring_stiffness="{joint_spring_stiffness}"/>
   </joint>
   <link
@@ -316,10 +323,10 @@
         value="0.0676525455789735" />
       <inertia
-        ixx="0.000122002023066796"
-        ixy="7.29593356230121E-13"
-        ixz="9.63170353371061E-09"
-        iyy="0.000122002023127152"
-        iyz="-9.24154949889042E-09"
-        izz="1.46043439809638E-12" />
+        ixx="0.001"
+        ixy="0"
+        ixz="0"
+        iyy="0.001"
+        iyz="0"
+        izz="0.001" />
     </inertial>
     <visual>
@@ -369,10 +376,10 @@
         value="0.0626921047058405" />
       <inertia
-        ixx="0.000115246639451415"
-        ixy="4.42139679831176E-14"
-        ixz="1.89711279909763E-09"
-        iyy="0.000115246639420046"
-        iyz="-2.68592949587539E-09"
-        izz="9.38270676408352E-14" />
+        ixx="0.001"
+        ixy="0"
+        ixz="0"
+        iyy="0.001"
+        iyz="0"
+        izz="0.001" />
     </inertial>
     <visual>
@@ -411,7 +418,8 @@
       link="link_arm_l3" />
     <axis
-	xyz="0 0 1" />
+  xyz="0 0 1" />
     <!-- 0.13 = 0.52/4-->
     <limit effort="100" lower="0.0" upper="0.13" velocity="1.0"/>
+    <dynamics damping="${joint_damping}" friction="${joint_friction}" spring_reference="${joint_spring_reference}" spring_stiffness="{joint_spring_stiffness}"/>
   </joint>
   <link
@@ -424,10 +432,10 @@
         value="0.0569074368576238" />
       <inertia
-        ixx="0.000105206697151872"
-        ixy="2.59896259031046E-14"
-        ixz="1.69941454517918E-09"
-        iyy="0.000105206697154717"
-        iyz="-1.60895568923743E-09"
-        izz="5.20570301686304E-14" />
+        ixx="0.001"
+        ixy="0"
+        ixz="0"
+        iyy="0.001"
+        iyz="0"
+        izz="0.001" />
     </inertial>
     <visual>
@@ -466,7 +474,8 @@
       link="link_arm_l2" />
     <axis
-	xyz="0 0 1" />
+  xyz="0 0 1" />
     <!-- 0.13 = 0.52/4-->
     <limit effort="100" lower="0.0" upper="0.13" velocity="1.0"/>
+    <dynamics damping="${joint_damping}" friction="${joint_friction}" spring_reference="${joint_spring_reference}" spring_stiffness="{joint_spring_stiffness}"/>
   </joint>
   <link
@@ -479,10 +488,10 @@
         value="0.0511763619538321" />
       <inertia
-        ixx="9.58490021274768E-05"
-        ixy="2.27446667584309E-14"
-        ixz="1.54951672295709E-09"
-        iyy="9.5849002131875E-05"
-        iyz="-1.40692486873422E-09"
-        izz="4.57014633924348E-14" />
+        ixx="0.001"
+        ixy="0"
+        ixz="0"
+        iyy="0.001"
+        iyz="0"
+        izz="0.001" />
     </inertial>
     <visual>
@@ -521,7 +530,8 @@
       link="link_arm_l1" />
     <axis
-	xyz="0 0 1" />
+  xyz="0 0 1" />
     <!-- 0.13 = 0.52/4-->
     <limit effort="100" lower="0.0" upper="0.13" velocity="1.0"/>
+    <dynamics damping="${joint_damping}" friction="${joint_friction}" spring_reference="${joint_spring_reference}" spring_stiffness="{joint_spring_stiffness}"/>
   </joint>
   <link
@@ -534,10 +544,10 @@
         value="0.101241250325294" />
       <inertia
-        ixx="0.000227156999010352"
-        ixy="8.90680620109423E-06"
-        ixz="-7.91132210985695E-05"
-        iyy="0.000300732790537324"
-        iyz="7.21771824540896E-06"
-        izz="9.35784422621597E-05" />
+        ixx="0.001"
+        ixy="0"
+        ixz="0"
+        iyy="0.001"
+        iyz="0"
+        izz="0.001" />
     </inertial>
     <visual>
@@ -576,7 +586,8 @@
       link="link_arm_l0" />
     <axis
-	xyz="0 0 1" />
+  xyz="0 0 1" />
     <!-- 0.13 = 0.52/4-->
     <limit effort="100" lower="0.0" upper="0.13" velocity="1.0"/>
+    <dynamics damping="${joint_damping}" friction="${joint_friction}" spring_reference="${joint_spring_reference}" spring_stiffness="{joint_spring_stiffness}"/>
   </joint>
   <link
@@ -589,10 +600,10 @@
         value="0.0405398981326229" />
       <inertia
-        ixx="2.20062857967227E-09"
-        ixy="1.15494401227051E-13"
-        ixz="1.02598056874346E-11"
-        iyy="2.20039759185237E-09"
-        iyz="-2.47692875363392E-11"
-        izz="3.26666802416509E-13" />
+        ixx="0.001"
+        ixy="0"
+        ixz="0"
+        iyy="0.001"
+        iyz="0"
+        izz="0.001" />
     </inertial>
     <visual>
@@ -607,5 +618,5 @@
         name="">
         <color
-	  rgba="0.792156862745098 0.819607843137255 0.933333333333333 1" />
+    rgba="0.792156862745098 0.819607843137255 0.933333333333333 1" />
       </material>
     </visual>
@@ -633,10 +644,11 @@
       xyz="0 0 -1" />
     <!--
-	stowed to front ~225 deg: 3.15159 x 1.25 = 3.9395
-	using 4.0
-	stowed to back ~100 deg:  100 / 180 x 3.14159 = 1.7453
-	using -1.75
+  stowed to front ~225 deg: 3.15159 x 1.25 = 3.9395
+  using 4.0
+  stowed to back ~100 deg:  100 / 180 x 3.14159 = 1.7453
+  using -1.75
     -->
     <limit effort="100" lower="-1.75" upper="4.0" velocity="1.0"/>
+    <dynamics damping="${joint_damping}" friction="${joint_friction}" spring_reference="${joint_spring_reference}" spring_stiffness="{joint_spring_stiffness}"/>
   </joint>
   <link
@@ -649,10 +661,10 @@
         value="0.129454717596498" />
       <inertia
-        ixx="2.9340596231093E-05"
-        ixy="-7.89638931853666E-07"
-        ixz="-4.74678128515878E-06"
-        iyy="2.68283736177377E-05"
-        iyz="1.80251508621876E-06"
-        izz="1.4617291423745E-05" />
+        ixx="0.001"
+        ixy="0"
+        ixz="0"
+        iyy="0.001"
+        iyz="0"
+        izz="0.001" />
     </inertial>
     <visual>
@@ -702,10 +714,10 @@
         value="0.035858341182617" />
       <inertia
-        ixx="2.75847937559827E-05"
-        ixy="5.25762707913649E-07"
-        ixz="-9.28796751052893E-07"
-        iyy="2.08815921106858E-05"
-        iyz="1.17265055331737E-05"
-        izz="6.78612505435872E-06" />
+        ixx="0.001"
+        ixy="0"
+        ixz="0"
+        iyy="0.001"
+        iyz="0"
+        izz="0.001" />
     </inertial>
     <visual>
@@ -744,6 +756,7 @@
       link="link_head_pan" />
     <axis
-	xyz="0 0 1" />
+  xyz="0 0 1" />
     <!-- unconstrained range for now -->
+    <dynamics damping="${joint_damping}" friction="${joint_friction}" spring_reference="${joint_spring_reference}" spring_stiffness="{joint_spring_stiffness}"/>
     <limit effort="100" lower="-3.9" upper="1.5" velocity="1.0"/>
   </joint>
@@ -757,10 +770,10 @@
         value="0.0701242408063442" />
       <inertia
-        ixx="1.73265934767466E-05"
-        ixy="2.38363792824069E-07"
-        ixz="7.96430204321056E-08"
-        iyy="4.11044416077217E-05"
-        iyz="-9.41955638215997E-07"
-        izz="2.38851808140542E-05" />
+        ixx="0.001"
+        ixy="0"
+        ixz="0"
+        iyy="0.001"
+        iyz="0"
+        izz="0.001" />
     </inertial>
     <visual>
@@ -801,4 +814,5 @@
       xyz="0 0 1" />
     <!-- unconstrained range for now -->
+    <dynamics damping="${joint_damping}" friction="${joint_friction}" spring_reference="${joint_spring_reference}" spring_stiffness="{joint_spring_stiffness}"/>
     <limit effort="100" lower="-1.53" upper="0.79" velocity="1.0"/>
   </joint>
