Commit message: Cleanup and complete xacro port

File: stretch_description/urdf/stretch_description.xacro (robot description, xacro)
@@ -1,4 +1,5 @@
 <?xml version="1.0"?>
 <robot xmlns:xacro="http://www.ros.org/wiki/xacro" name="stretch_description">
+  <xacro:arg name="realsense" default="true"/>
   <xacro:include filename="stretch_gripper.xacro" />
   <!--<xacro:include filename="stretch_gripper_with_puller.xacro" />-->
@@ -6,6 +7,8 @@
   <xacro:include filename="stretch_main.xacro" />
   <xacro:include filename="stretch_aruco.xacro" />
-  <xacro:include filename="stretch_d435i.xacro" />
   <xacro:include filename="stretch_laser_range_finder.xacro" />
   <xacro:include filename="stretch_respeaker.xacro" />
+  <xacro:if value="$(arg realsense)">
+    <xacro:include filename="stretch_d435i.xacro" />
+  </xacro:if>
 </robot>

File: stretch_description/urdf/stretch_gripper.xacro (robot description, xacro)
@@ -2,6 +2,6 @@
 <robot xmlns:xacro="http://www.ros.org/wiki/xacro" name="stretch_gripper">
   <xacro:property name="scale_finger_length" value="0.9" />
-  <xacro:property name="gripper_joint_damping" value="0.75"/>
-  <xacro:property name="gripper_joint_friction" value="2.48"/>
+  <xacro:property name="gripper_joint_damping" value="5.75"/>
+  <xacro:property name="gripper_joint_friction" value="5.48"/>
   <xacro:property name="gripper_joint_spring_stiffness" value="0"/>
   <xacro:property name="gripper_joint_spring_reference" value="0"/>
@@ -104,5 +104,5 @@
     <dynamics damping="${gripper_joint_damping}" friction="${gripper_joint_friction}" spring_reference="${gripper_joint_spring_reference}" spring_stiffness="{gripper_joint_spring_stiffness}"/>
   </joint>
-  <link
+  <!-- <link
     name="link_gripper_fingertip_left">
     <inertial>
@@ -151,5 +151,5 @@
     <axis
       xyz="0 0 0" />
-  </joint>
+  </joint> -->
   <link
     name="link_gripper_finger_right">
@@ -202,5 +202,5 @@
     <dynamics damping="${gripper_joint_damping}" friction="${gripper_joint_friction}" spring_reference="${gripper_joint_spring_reference}" spring_stiffness="{gripper_joint_spring_stiffness}"/>
   </joint>
-  <link
+  <!-- <link
     name="link_gripper_fingertip_right">
     <inertial>
@@ -249,5 +249,5 @@
     <axis
       xyz="0 0 0" />
-  </joint>
+  </joint> -->
   <link
       name="link_grasp_center">

File: stretch_description/urdf/stretch_ignition_plugins.xacro (robot description, xacro)
@@ -14,4 +14,98 @@
       <frame_id>odom</frame_id>
       <child_frame_id>base_link</child_frame_id>
+    </plugin>
+    <!-- Joint Trajectories -->
+    <plugin filename="libignition-gazebo-joint-trajectory-controller-system.so" name="ignition::gazebo::systems::JointTrajectoryController">
+      <topic>joint_trajectory</topic>
+      <joint_name>joint_arm_l0</joint_name>
+      <initial_position>0</initial_position>
+      <position_p_gain>3000</position_p_gain>
+      <position_d_gain>15</position_d_gain>
+      <position_i_gain>1650</position_i_gain>
+      <position_i_min>-15</position_i_min>
+      <position_i_max>15</position_i_max>
+      <position_cmd_min>-87</position_cmd_min>
+      <position_cmd_max>87</position_cmd_max>
+      <joint_name>joint_arm_l1</joint_name>
+      <initial_position>0</initial_position>
+      <position_p_gain>3000</position_p_gain>
+      <position_d_gain>15</position_d_gain>
+      <position_i_gain>1650</position_i_gain>
+      <position_i_min>-15</position_i_min>
+      <position_i_max>15</position_i_max>
+      <position_cmd_min>-87</position_cmd_min>
+      <position_cmd_max>87</position_cmd_max>
+      <joint_name>joint_arm_l2</joint_name>
+      <initial_position>0</initial_position>
+      <position_p_gain>3000</position_p_gain>
+      <position_d_gain>15</position_d_gain>
+      <position_i_gain>1650</position_i_gain>
+      <position_i_min>-15</position_i_min>
+      <position_i_max>15</position_i_max>
+      <position_cmd_min>-87</position_cmd_min>
+      <position_cmd_max>87</position_cmd_max>
+      <joint_name>joint_arm_l3</joint_name>
+      <initial_position>0</initial_position>
+      <position_p_gain>3000</position_p_gain>
+      <position_d_gain>15</position_d_gain>
+      <position_i_gain>1650</position_i_gain>
+      <position_i_min>-15</position_i_min>
+      <position_i_max>15</position_i_max>
+      <position_cmd_min>-87</position_cmd_min>
+      <position_cmd_max>87</position_cmd_max>
+      <joint_name>joint_lift</joint_name>
+      <initial_position>0</initial_position>
+      <position_p_gain>3000</position_p_gain>
+      <position_d_gain>15</position_d_gain>
+      <position_i_gain>1650</position_i_gain>
+      <position_i_min>-15</position_i_min>
+      <position_i_max>15</position_i_max>
+      <position_cmd_min>-87</position_cmd_min>
+      <position_cmd_max>87</position_cmd_max>
+      <joint_name>joint_wrist_yaw</joint_name>
+      <initial_position>0</initial_position>
+      <position_p_gain>3000</position_p_gain>
+      <position_d_gain>15</position_d_gain>
+      <position_i_gain>1650</position_i_gain>
+      <position_i_min>-15</position_i_min>
+      <position_i_max>15</position_i_max>
+      <position_cmd_min>-87</position_cmd_min>
+      <position_cmd_max>87</position_cmd_max>
+      <joint_name>joint_gripper_finger_left</joint_name>
+      <initial_position>0</initial_position>
+      <position_p_gain>3000</position_p_gain>
+      <position_d_gain>15</position_d_gain>
+      <position_i_gain>1650</position_i_gain>
+      <position_i_min>-15</position_i_min>
+      <position_i_max>15</position_i_max>
+      <position_cmd_min>-87</position_cmd_min>
+      <position_cmd_max>87</position_cmd_max>
+      <joint_name>joint_gripper_finger_right</joint_name>
+      <initial_position>0</initial_position>
+      <position_p_gain>3000</position_p_gain>
+      <position_d_gain>15</position_d_gain>
+      <position_i_gain>1650</position_i_gain>
+      <position_i_min>-15</position_i_min>
+      <position_i_max>15</position_i_max>
+      <position_cmd_min>-87</position_cmd_min>
+      <position_cmd_max>87</position_cmd_max>
+      <joint_name>joint_head_pan</joint_name>
+      <initial_position>0</initial_position>
+      <position_p_gain>300</position_p_gain>
+      <position_d_gain>2.9</position_d_gain>
+      <position_i_gain>10</position_i_gain>
+      <position_i_min>-15</position_i_min>
+      <position_i_max>15</position_i_max>
+      <position_cmd_min>-50</position_cmd_min>
+      <position_cmd_max>50</position_cmd_max>
+      <joint_name>joint_head_tilt</joint_name>
+      <initial_position>0</initial_position>
+      <position_p_gain>300</position_p_gain>
+      <position_d_gain>2.9</position_d_gain>
+      <position_i_gain>10</position_i_gain>
+      <position_i_min>-15</position_i_min>
+      <position_i_max>15</position_i_max>
+      <position_cmd_min>-50</position_cmd_min>
+      <position_cmd_max>50</position_cmd_max>
     </plugin>
   </gazebo>
@@ -45,4 +139,8 @@
           <resolution>0.01</resolution>
         </range>
+        <noise type="gaussian">
+          <mean>0.0</mean>
+          <stddev>0.001</stddev>
+        </noise>
       </lidar>
       <alwaysOn>1</alwaysOn>
@@ -50,17 +148,61 @@
     </sensor>
   </gazebo>
-  <!-- TODO: Tune Sensors -->
   <gazebo reference="base_link">
     <!-- Base IMU (Accel + Gyro) -->
     <sensor name="imu" type="imu">
       <always_on>1</always_on>
-      <update_rate>100</update_rate>
+      <update_rate>25</update_rate>
       <visualize>false</visualize>
       <topic>imu</topic>
+      <imu>
+        <!-- 0.0625/2000 -->
+        <angular_velocity>
+          <x>
+            <noise type="gaussian">
+              <mean>0.0</mean>
+              <stddev>0.00003125</stddev>
+            </noise>
+          </x>
+          <y>
+            <noise type="gaussian">
+              <mean>0.0</mean>
+              <stddev>0.00003125</stddev>
+            </noise>
+          </y>
+          <z>
+            <noise type="gaussian">
+              <mean>0.0</mean>
+              <stddev>0.00003125</stddev>
+            </noise>
+          </z>
+        </angular_velocity>
+        <!-- 20/2000 noise -->
+        <linear_acceleration>
+          <x>
+            <noise type="gaussian">
+              <mean>0.0</mean>
+              <stddev>0.01</stddev>
+            </noise>
+          </x>
+          <y>
+            <noise type="gaussian">
+              <mean>0.0</mean>
+              <stddev>0.01</stddev>
+            </noise>
+          </y>
+          <z>
+            <noise type="gaussian">
+              <mean>0.0</mean>
+              <stddev>0.01</stddev>
+            </noise>
+          </z>
+        </linear_acceleration>
+      </imu>
     </sensor>
     <!-- Base Mag -->
+    <!-- 10/1200 noise -->
     <sensor name="magnetometer" type="magnetometer">
       <always_on>1</always_on>
-      <update_rate>100</update_rate>
+      <update_rate>25</update_rate>
       <visualize>false</visualize>
       <topic>magnetometer</topic>
@@ -69,5 +211,5 @@
           <noise type="gaussian">
             <mean>0.0</mean>
-            <stddev>0.1</stddev>
+            <stddev>0.0083</stddev>
           </noise>
         </x>
@@ -75,5 +217,5 @@
           <noise type="gaussian">
             <mean>0.0</mean>
-            <stddev>0.1</stddev>
+            <stddev>0.0083</stddev>
           </noise>
         </y>
@@ -81,5 +223,5 @@
           <noise type="gaussian">
             <mean>0.0</mean>
-            <stddev>0.1</stddev>
+            <stddev>0.0083</stddev>
           </noise>
         </z>
@@ -87,4 +229,5 @@
     </sensor>
   </gazebo>
+  <!-- TODO: Make this accelerometer only -->
   <!-- Wrist IMU (Accel Only) -->
   <gazebo reference="link_wrist_yaw">
@@ -94,7 +237,51 @@
       <visualize>false</visualize>
       <topic>wrist_imu</topic>
+      <imu>
+        <angular_velocity>
+          <x>
+            <noise type="gaussian">
+              <mean>0.0</mean>
+              <stddev>0.0</stddev>
+            </noise>
+          </x>
+          <y>
+            <noise type="gaussian">
+              <mean>0.0</mean>
+              <stddev>0.0</stddev>
+            </noise>
+          </y>
+          <z>
+            <noise type="gaussian">
+              <mean>0.0</mean>
+              <stddev>0.0</stddev>
+            </noise>
+          </z>
+        </angular_velocity>
+        <!-- 1.1/2000 Noise -->
+        <linear_acceleration>
+          <x>
+            <noise type="gaussian">
+              <mean>0.0</mean>
+              <stddev>0.00055</stddev>
+            </noise>
+          </x>
+          <y>
+            <noise type="gaussian">
+              <mean>0.0</mean>
+              <stddev>0.00055</stddev>
+            </noise>
+          </y>
+          <z>
+            <noise type="gaussian">
+              <mean>0.0</mean>
+              <stddev>0.00055</stddev>
+            </noise>
+          </z>
+        </linear_acceleration>
+      </imu>
     </sensor>
   </gazebo>
   <!-- Realsense IMU -->
+  <xacro:if value="$(arg realsense)">
   <gazebo reference="camera_joint">
     <preserveFixedJoint>true</preserveFixedJoint>
@@ -107,4 +294,5 @@
   </gazebo>
   <gazebo reference="camera_gyro_frame">
+    <!-- Arbitrary noise -->
     <sensor name="realsense_imu" type="imu">
       <always_on>1</always_on>
@@ -112,4 +300,46 @@
       <visualize>false</visualize>
       <topic>realsense_imu</topic>
+      <imu>
+        <angular_velocity>
+          <x>
+            <noise type="gaussian">
+              <mean>0.0</mean>
+              <stddev>0.001</stddev>
+            </noise>
+          </x>
+          <y>
+            <noise type="gaussian">
+              <mean>0.0</mean>
+              <stddev>0.001</stddev>
+            </noise>
+          </y>
+          <z>
+            <noise type="gaussian">
+              <mean>0.0</mean>
+              <stddev>0.001</stddev>
+            </noise>
+          </z>
+        </angular_velocity>
+        <linear_acceleration>
+          <x>
+            <noise type="gaussian">
+              <mean>0.0</mean>
+              <stddev>0.001</stddev>
+            </noise>
+          </x>
+          <y>
+            <noise type="gaussian">
+              <mean>0.0</mean>
+              <stddev>0.001</stddev>
+            </noise>
+          </y>
+          <z>
+            <noise type="gaussian">
+              <mean>0.0</mean>
+              <stddev>0.001</stddev>
+            </noise>
+          </z>
+        </linear_acceleration>
+      </imu>
     </sensor>
   </gazebo>
@@ -123,7 +353,7 @@
   <gazebo reference="camera_color_optical_frame">
     <sensor name="realsense_d435_color" type="camera">
-      <update_rate>60</update_rate>
+      <update_rate>30</update_rate>
       <camera name="camera">
-        <horizontal_fov>1.0472</horizontal_fov>
+        <horizontal_fov>1.13446</horizontal_fov>
         <lens>
           <intrinsics>
@@ -170,7 +400,7 @@
   <gazebo reference="camera_depth_optical_frame">
     <sensor name="realsense_d435" type="rgbd_camera">
-      <update_rate>60</update_rate>
+      <update_rate>30</update_rate>
       <camera name="camera">
-        <horizontal_fov>1.0472</horizontal_fov>
+        <horizontal_fov>1.13446</horizontal_fov>
         <lens>
           <intrinsics>
@@ -222,7 +452,7 @@
   <gazebo reference="camera_infra1_optical_frame">
     <sensor name="realsense_d435_ir" type="camera">
-      <update_rate>60</update_rate>
+      <update_rate>30</update_rate>
       <camera name="camera">
-        <horizontal_fov>1.0472</horizontal_fov>
+        <horizontal_fov>1.13446</horizontal_fov>
         <lens>
           <intrinsics>
@@ -268,7 +498,7 @@
   <gazebo reference="camera_infra2_optical_frame">
     <sensor name="realsense_d435_ir2" type="camera">
-      <update_rate>60</update_rate>
+      <update_rate>30</update_rate>
       <camera name="camera">
-        <horizontal_fov>1.0472</horizontal_fov>
+        <horizontal_fov>1.13446</horizontal_fov>
         <lens>
           <intrinsics>
@@ -305,3 +535,4 @@
     </sensor>
   </gazebo>
+</xacro:if>
 </robot>

File: stretch_description/urdf/stretch_main.xacro (robot description, xacro)
@@ -2,6 +2,6 @@
 <robot xmlns:xacro="http://www.ros.org/wiki/xacro" name="stretch_main">
   <xacro:property name="M_PI" value="3.1415926535897931" />
-  <xacro:property name="joint_damping" value="0.75"/>
-  <xacro:property name="joint_friction" value="2.48"/>
+  <xacro:property name="joint_damping" value="21.75"/>
+  <xacro:property name="joint_friction" value="10.48"/>
   <xacro:property name="joint_spring_stiffness" value="0"/>
   <xacro:property name="joint_spring_reference" value="0"/>
@@ -142,5 +142,4 @@
       xyz="0 0 1" />
       <dynamics damping="${joint_damping}" friction="${joint_friction}" spring_reference="${joint_spring_reference}" spring_stiffness="{joint_spring_stiffness}"/>
-      <!-- <dynamics damping="21.75" friction="3.48" spring_reference="0.0" spring_stiffness="0.0"/> -->
   </joint>
   <!-- Representing a ball joint -->
