Commit message: New demo package and general improvements on stretch

File: stretch_description/urdf/stretch_ignition_plugins.xacro (robot description, xacro)
@@ -2,4 +2,12 @@
 <robot xmlns:xacro="http://www.ros.org/wiki/xacro" name="stretch_description">
   <gazebo>
+    <!-- Odometry Publisher -->
+    <plugin filename="ignition-gazebo-odometry-publisher-system" name="ignition::gazebo::systems::OdometryPublisher">
+      <odom_publish_frequency>50</odom_publish_frequency>
+      <odom_topic>/odom</odom_topic>
+      <odom_frame>odom</odom_frame>
+      <robot_base_frame>base_link</robot_base_frame>
+      <dimensions>3</dimensions>
+    </plugin>
     <!-- Joint States -->
     <plugin filename="libignition-gazebo-joint-state-publisher-system.so" name="ignition::gazebo::systems::JointStatePublisher"/>
@@ -12,5 +20,5 @@
       <odom_publish_frequency>10</odom_publish_frequency>
       <topic>cmd_vel</topic>
-      <frame_id>odom</frame_id>
+      <frame_id>diff_odom</frame_id>
       <child_frame_id>base_link</child_frame_id>
     </plugin>
@@ -374,6 +382,6 @@
         </distortion>
         <image>
-          <width>1920</width>
-          <height>1080</height>
+          <width>640</width>
+          <height>480</height>
           <format>R8G8B8</format>
         </image>

File: stretch_description/urdf/stretch_main.xacro (robot description, xacro)
@@ -144,5 +144,5 @@
   </joint>
   <!-- Representing a ball joint -->
-  <joint name="caster_joint_theta" type="continuous">
+  <!-- <joint name="caster_joint_theta" type="continuous">
     <origin xyz="-0.245 0.0 0.032" rpy="${-M_PI/2} 0 0"/>
     <parent link="base_link"/>
@@ -183,5 +183,5 @@
       <limit lower="${-pi/2}" upper="${-pi/2}" velocity="${caster_velocity_limit}" effort="${caster_effort_limit}" />
     </inertial>
-  </link>
+  </link> -->
   <link name="link_caster">
     <collision>
@@ -232,8 +232,8 @@
   </link>
   <joint name="joint_caster" type="fixed">
-    <parent link="caster_link_phi"/>
-    <!-- <parent link="base_link"/> -->
+    <!-- <parent link="caster_link_phi"/> -->
+    <parent link="base_link"/>
     <child link="link_caster"/>
-    <!-- <origin xyz="-0.245 0.0 0.032" rpy="${-M_PI/2} 0 0"/> -->
+    <origin xyz="-0.245 0.0 0.032" rpy="${-M_PI/2} 0 0"/>
   </joint>
   <link
